File: Eagle/mk2.sch (EAGLE design)
At the start: 87 parts, among them Q1 BC847B, SW1 EVQQ2, SW2 MFP106D, U1 TPS63061DSCT, U2 TPS63061DSCT, U3 DRV8833PWPR, U4 TCA9406DCTR, U5 MPU-6050, U6 74AHCT1G32GW/T1, U7 ATMEGA328-AU

Commit message: update
files
Parts:
- removed BUZ1: KSSG74B16, Jaegger_MKII:KSSG74B16
- removed D1: S1B-13-F, Jaegger_MKII:S1B-13-F
- removed JP6, JP7: (no value), pinhead:PINHD-1X2
- removed R14, R15: 10k, resistor:R-EU_R0805
- added BLUETOOTH1: HC-06 Female Header, pinhead:PINHD-1X4
- added BUZZ1: KTG1205C, Jaegger_MKII:KTG1205C
- added C20, C21: 0.1µF, rcl:C-EUC0805
- added IR_REC1, IR_REC2, IR_REC3, IR_REC4: TSMP77000TR, Jaegger_MKII:TSMP77000TR
- added R16: 10k, rcl:R-EU_R0805
- added R17, R18: 1k, rcl:R-EU_R0805
- added R20, R21: 20KOHM, Panasonic-Trimmer_Potentiometers:EVM2NSX80B24-2N
- added U$1, U$2: KPA-3010F3C, Jaegger_MKII:KPA-3010F3C
- added U11: UA555D, linear:UA555D
- added U8: 74ALS08D, 74xx-eu:74ALS08D
- C10: value 0.1µF -> 2.2nF; device rcl:C-EUC0805K -> rcl:C-EUC0805
- C19: value 2.2nF -> 0.1µF
- C7: value 0.1uF -> 0.1µF
- C9: device rcl:C-EUC0805K -> rcl:C-EUC0805
- FRONT_IR_SENSOR: device pinhead:PINHD-1X6 -> pinhead:PINHD-1X8
- JP1: value Arduino Leonardo -> (none); device pinhead:PINHD-1X8 -> pinhead:PINHD-1X17
- JP2: value Arduino Leonardo -> (none); device pinhead:PINHD-1X10 -> pinhead:PINHD-1X17
- JP3: value Arduino Leonardo -> IR1; device pinhead:PINHD-1X8 -> pinhead:PINHD-1X3
- JP4: value Arduino Leonardo -> IR2; device pinhead:PINHD-1X6 -> pinhead:PINHD-1X3
- R10, R11, R8, R9: value 330 -> 1k
- R2: value 330 -> 10k
- U4: device texas:TCA9406DCTR -> TCA9406DCTR:TCA9406DCTR
- renumbered IR1 to AN1, IR2 to AN2
Connections:
- net ADC6 renamed ADC6_EXT
- net ADC7 renamed ADC7_EXT
- removed net AN3: U7.PC3_(ADC3/PCINT11)
- removed net BUTTON: JP3.6, SW1.P$1
- removed net BUZZER_ARDUINO: JP2.6, U6.A
- removed net CAÑON: D4.1, JP3.4
- removed net ECHO_ARDUINO: JP3.1, ULTRASONIC1.3
- removed net ILUM_3: LED8.A, U7.(PCINT2/SS/OC1B)_PB2
- removed net ILUM_4: LED9.A, U7.PC2_(ADC2/PCINT10)
- removed net MISO: ICSP.1, U7.(PCINT4/MISO)_PB4
- removed net SERVO1: D13~.1, JP2.5
- removed net SERVO2: D5~.1, JP3.3
- removed net TRIGGER_ARDUINO: JP2.10, ULTRASONIC1.2
- new net BUTTON/D16/328: JP1.1, R2.2, SW1.P$2, U7.PC3_(ADC3/PCINT11)
- new net D10/BIN2: JP1.15, U8B.I0
- new net D11/BIN1: JP1.16, U8A.I0
- new net D12/BUZZER_ARDUINO: JP1.17, R16.1, U6.A
- new net D13/SERVO1: D13~.1, JP2.17
- new net D14/MISO_MICRO: IR_REC1.C_OUT, JP2.2
- new net D15/SCK_MICRO: IR_REC2.C_OUT, JP2.1
- new net D4/CAÑON: D4.1, JP1.9
- new net D5/SERVO2: D5~.1, JP1.10
- new net D6/AIN2: JP1.11, U8D.I0
- new net D7/ECHO_ARDUINO: JP1.12, JP4.1, ULTRASONIC1.3
- new net D8/TRIGGER_ARDUINO: JP1.13, JP3.1, ULTRASONIC1.2
- new net D9/AIN1: JP1.14, U8C.I0
- new net ILUM1: U7.(PCINT2/SS/OC1B)_PB2
- new net MISO/IR_REAR_LEFT: BACK_IR_SENSOR.4, ICSP.1, U7.(PCINT4/MISO)_PB4
- new net MOSI/ENABLE: U7.(PCINT3/OC2A/MOSI)_PB3, U8A.I1, U8B.I1, U8C.I1, U8D.I1
- new net N$35: C10.1, U5.CPOUT
- new net N$36: C9.1, U5.REGOUT
- new net N$39: R20.3, R21.2, U11.DIS
- new net N$40: R18.1, U$2.C
- new net N$42: C21.1, U11.CV
- new net OUTPUT_555: U$1.A, U$2.A, U11.Q
- new net RX328: BLUETOOTH1.3, U7.PD0_(RXD/PCINT16)
- new net SCK/IR_REAR_RIGHT: U7.PB5_(SCK/PCINT5)
- new net TX328/ENABLE555: BLUETOOTH1.4, U11.R, U7.PD1_(TXD/PCINT17)
- net +3V3: now also JP2.16; no longer C10.1, C7.1, JP1.4, U5.VDD, U5.VLOGIC
- net +5V_CONTROL: now also BLUETOOTH1.1, BUZZ1.+, C7.1, C8.1, IR_REC1.VS, IR_REC2.VS, IR_REC3.VS, IR_REC4.VS, JP2.3, JP2.6, JP3.2, JP4.2, R2.1, R20.2, U11.V+, U8P.VCC; no longer BUZ1.2, C9.1, D1.2, JP1.5, JP1.8, JP6.1, JP7.1
- net A0: now also FRONT_IR_SENSOR.1, JP2.14; no longer FRONT_IR_SENSOR.6, JP4.1
- net A1: now also FRONT_IR_SENSOR.2, JP2.13; no longer FRONT_IR_SENSOR.5, JP4.2
- net A2: now also FRONT_IR_SENSOR.3, JP2.12; no longer FRONT_IR_SENSOR.2, JP4.3
- net A3: now also FRONT_IR_SENSOR.6, JP2.11; no longer FRONT_IR_SENSOR.1, JP4.4
- net A4: now also FRONT_IR_SENSOR.7, JP2.10; no longer BACK_IR_SENSOR.4, JP4.5
- net A5: now also FRONT_IR_SENSOR.8, JP2.9; no longer BACK_IR_SENSOR.1, JP4.6
- net AIN1: now also U8C.O; no longer JP2.9
- net AIN2: now also U8D.O; no longer JP3.2
- net BIN1: now also U8A.O; no longer JP2.7
- net BIN2: now also U8B.O; no longer JP2.8
- net D0/RX: now also JP1.4; no longer JP3.8
- net D1/TX: now also JP1.3; no longer JP3.7
- net DEBIL_1: now also IR_REC3.C_OUT; no longer JP7.2, R15.2
- net DEBIL_2: now also IR_REC4.C_OUT; no longer JP6.2, R14.2
- net GND: now also BLUETOOTH1.2, C20.2, C21.2, FRONT_IR_SENSOR.5, IR_REC1.GND@1, IR_REC1.GND@2, IR_REC2.GND@1, IR_REC2.GND@2, IR_REC3.GND@1, IR_REC3.GND@2, IR_REC4.GND@1, IR_REC4.GND@2, JP3.3, JP4.3, R16.2, R17.2, R18.2, SW1.P$1, U11.GND, U8P.GND; no longer FRONT_IR_SENSOR.3, JP1.7, R14.1, R15.1, R2.1, U5.CLKIN
- net ILUM_1: now also LED7.A; no longer U7.(PCINT21/OC0B/T1)_PD5
- net ILUM_2: now also LED8.A, LED9.A, U7.PC2_(ADC2/PCINT10); no longer LED7.A, U7.(PCINT22/OC0A/AIN0)_PD6
- net MOSI: no longer U7.(PCINT3/OC2A/MOSI)_PB3
- net N$17: now also BUZZ1.-; no longer BUZ1.1, D1.1
- net N$23: now also R17.1, U$1.C; no longer R2.2, SW1.P$2
- net N$31: now also C20.1, R21.3, U11.THR, U11.TR; no longer C8.1, U5.REGOUT
- net N$5: now also U5.VDD, U5.VLOGIC; no longer U5.CPOUT
- net SCK: now also BACK_IR_SENSOR.1; no longer U7.PB5_(SCK/PCINT5)
- net SCL_5: now also JP1.8; no longer JP2.1
- net SDA_5: now also JP1.7; no longer JP2.2
- net VIDA_1: now also U7.PD2_(INT0/PCINT18); no longer U7.PD0_(RXD/PCINT16)
- net VIDA_2: now also U7.(PCINT19/OC2B/INT1)_PD3; no longer U7.PD1_(TXD/PCINT17)
- net VIDA_3: now also U7.(PCINT20/XCK/T0)_PD4; no longer U7.PD2_(INT0/PCINT18)
- net VIDA_4: now also U7.(PCINT21/OC0B/T1)_PD5; no longer U7.(PCINT19/OC2B/INT1)_PD3
- net VIDA_5: now also U7.(PCINT22/OC0A/AIN0)_PD6; no longer U7.(PCINT20/XCK/T0)_PD4
Other:
- moved on the sheet: 3,3V, 5V_CONTROL, 5V_SERVO, BACK_IR_SENSOR, C1, C10, C18, C19, C2, C3, C4, C5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
