File: Eagle/MainBoard/mk2.sch (EAGLE design)
At the start: 98 parts, among them Q1 BC847B, SW1 EVQQ2, SW2 MFP106D, U1 TPS63061DSCT, U11 UA555D, U2 TPS63061DSCT, U3 DRV8833PWPR, U4 TCA9406DCTR, U5 MPU-6050, U6 74AHCT1G32GW/T1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

Commit message: Update
Parts:
- added F1: (no value), rcl:R-EU_R1206
- renumbered U$1 to D1, U$2 to D2, U11 to U9
Connections:
- net N$37 renamed BM1
- net N$38 renamed AM1
- net N$40 renamed D2
- removed net MOSI: ICSP.4
- removed net SCK: BACK_IR_SENSOR.1, ICSP.3
- new net N$41: F1.2, SW2.COM
- net MOSI/ENABLE: now also ICSP.4
- net N$6: now also F1.1; no longer SW2.COM
- net SCK/IR_REAR_RIGHT: now also BACK_IR_SENSOR.1, ICSP.3
Other:
- moved on the sheet: SW2
